Commit message: start adding pieces to the visualization of the hand with fingers

File: ur_e_description/urdf/ur5e.urdf.xacro (robot description, xacro)
@@ -278,4 +278,80 @@
       </xacro:cylinder_inertial>
     </link>
+    <link name="${prefix}wrist_coupling_link">
+      <visual>
+        <geometry>
+          <mesh filename="package://ur_e_description/meshes/ur5e/visual/wrist_coupling.STL" />
+        </geometry>
+        <material name="LightGrey">
+          <color rgba="0.7 0.7 0.7 1.0"/>
+        </material>
+      </visual>
+      <collision>
+        <geometry>
+          <mesh filename="package://ur_e_description/meshes/ur5e/visual/wrist_coupling.STL" />
+        </geometry>
+      </collision>
+      <!-- computed from https://robotiq.com/support/hand-e-adaptive-robot-gripper/documents-gripper-instruction-manual-e-series weight was guessed -->
+      <xacro:cylinder_inertial radius="0.375" length="0.0169" mass="0.010">
+        <origin xyz="0.0 0.0 0.0" rpy="0 0 0" />
+      </xacro:cylinder_inertial>
+    </link>
+    <joint name="${prefix}wrist_coupling_fixed_joint" type="fixed">
+      <parent link="${prefix}wrist_3_link" />
+      <child link = "${prefix}wrist_coupling_link" />
+      <!-- will need to fudge the length to account for origin being inside the coupling -->
+      <origin xyz="0.0 ${wrist_3_length} 0.0" rpy="${-pi/2.0} 0.0 0.0" />
+    </joint>
+    <link name="${prefix}hand_link">
+      <visual>
+        <geometry>
+          <mesh filename="package://ur_e_description/meshes/ur5e/visual/robotiq_hand_e.STL" />
+        </geometry>
+        <material name="LightGrey">
+          <color rgba="0.7 0.7 0.7 1.0"/>
+        </material>
+      </visual>
+      <collision>
+        <geometry>
+          <mesh filename="package://ur_e_description/meshes/ur5e/visual/robotiq_hand_e.STL" />
+        </geometry>
+      </collision>
+      <!-- pulled from https://robotiq.com/support/hand-e-adaptive-robot-gripper/documents-gripper-instruction-manual-e-series -->
+      <inertial>
+        <mass value="1.090"/>
+        <inertia ixx="0.005341" ixy="0" ixz="0" iyy="0.005447" iyz="0" izz="0.000636"/>
+        <origin xyz="0.0 0.0 0.0575" rpy="0.0 0.0 0.0" />
+      </inertial>
+    </link>
+    <joint name="${prefix}hand_coupling_fixed_joint" type="fixed">
+      <parent link="${prefix}wrist_coupling_link" />
+      <child link = "${prefix}hand_link" />
+      <!-- we fudge the length to make the two line up (probably because origin of hand is in rando place -->
+      <origin xyz="0.0 0.0 ${0.1005 - 0.0075}" rpy="${pi/2.0} 0.0 ${pi/2.0}" />
+    </joint>
+    <link name="${prefix}finger_l_link">
+      <visual>
+        <geometry>
+          <mesh filename="package://ur_e_description/meshes/ur5e/visual/hand_e_finger.STL" />
+        </geometry>
+        <material name="LightGrey">
+          <color rgba="0.7 0.7 0.7 1.0"/>
+        </material>
+      </visual>
+      <collision>
+        <geometry>
+          <mesh filename="package://ur_e_description/meshes/ur5e/visual/hand_e_finger.STL" />
+        </geometry>
+      </collision>
+      <!-- lazy guess -->
+      <xacro:cylinder_inertial radius="0.005" length="0.01" mass="0.001">
+        <origin xyz="0.0 0.0 0.0" rpy="0 0 0" />
+      </xacro:cylinder_inertial>
+    </link>
+    <joint name="${prefix}finger_l_fixed_joint" type="fixed">
+      <parent link="${prefix}hand_link" />
+      <child link = "${prefix}finger_l_link" />
+      <origin xyz="0.0 0.0 0.0" rpy="0.0 0.0 0.0" />
+    </joint>
     <joint name="${prefix}ee_fixed_joint" type="fixed">
       <parent link="${prefix}wrist_3_link" />
@@ -291,4 +367,27 @@
       </collision>
     </link>
+    <link name="${prefix}camera_holder">
+      <visual>
+        <geometry>
+          <mesh filename="package://ur_e_description/meshes/ur5e/visual/camera_mount_v2.STL" />
+        </geometry>
+        <material name="LightGrey">
+          <color rgba="0.7 0.7 0.7 1.0"/>
+        </material>
+      </visual>
+      <collision>
+        <geometry>
+          <mesh filename="package://ur_e_description/meshes/ur5e/visual/camera_mount_v2.STL" />
+        </geometry>
+      </collision>
+      <xacro:cylinder_inertial radius="0.6" length="0.12" mass="0.01">
+        <origin xyz="0.0 0.0 0.0" rpy="0 0 0" />
+      </xacro:cylinder_inertial>
+    </link>
+    <joint name="${prefix}camera_holder_fixed_joint" type="fixed">
+      <parent link="${prefix}wrist_3_link" />
+      <child link = "${prefix}camera_holder" />
+      <origin xyz="0.0 0.0 0.0" rpy="0.0 0.0 0.0" />
+    </joint>
     <xacro:ur_arm_transmission prefix="${prefix}" />
     <xacro:ur_arm_gazebo prefix="${prefix}" />

Commit message: making such a pretty robot example

File: ur_e_description/urdf/ur5e.urdf.xacro (robot description, xacro)
@@ -349,8 +349,32 @@
       </xacro:cylinder_inertial>
     </link>
+    <link name="${prefix}finger_r_link">
+      <visual>
+        <geometry>
+          <mesh filename="package://ur_e_description/meshes/ur5e/visual/hand_e_finger.STL" />
+        </geometry>
+        <material name="LightGrey">
+          <color rgba="0.7 0.7 0.7 1.0"/>
+        </material>
+      </visual>
+      <collision>
+        <geometry>
+          <mesh filename="package://ur_e_description/meshes/ur5e/visual/hand_e_finger.STL" />
+        </geometry>
+      </collision>
+      <!-- lazy guess -->
+      <xacro:cylinder_inertial radius="0.005" length="0.01" mass="0.001">
+        <origin xyz="0.0 0.0 0.0" rpy="0 0 0" />
+      </xacro:cylinder_inertial>
+    </link>
     <joint name="${prefix}finger_l_fixed_joint" type="fixed">
       <parent link="${prefix}hand_link" />
       <child link = "${prefix}finger_l_link" />
-      <origin xyz="0.0 0.0 0.0" rpy="0.0 0.0 0.0" />
+      <origin xyz="0.0 ${0.046 + 0.015} 0.0" rpy="0.0 0.0 ${-pi/2.0}" />
+    </joint>
+    <joint name="${prefix}finger_r_fixed_joint" type="fixed">
+      <parent link="${prefix}hand_link" />
+      <child link = "${prefix}finger_r_link" />
+      <origin xyz="0.0 ${0.046 + 0.015} 0.0" rpy="${pi} 0.0 ${-pi/2.0}" />
     </joint>
     <joint name="${prefix}ee_fixed_joint" type="fixed">

Commit message: set to ur5 EEEE and add tool tip frame

File: ur_e_description/urdf/ur5e.urdf.xacro (robot description, xacro)
@@ -330,4 +330,10 @@
       <origin xyz="0.0 0.0 ${0.1005 - 0.0075}" rpy="${pi/2.0} 0.0 ${pi/2.0}" />
     </joint>
+    <link name="${prefix}grasp_point_fixed"/>
+    <joint name="${prefix}grasp_point_fixed_joint" type="fixed">
+      <parent link="${prefix}hand_link" />
+      <child link = "${prefix}grasp_point_fixed" />
+      <origin xyz="0.0 0.0 0.050" rpy="0.0 0.0 0.0" />
+    </joint>
     <link name="${prefix}finger_l_link">
       <visual>

Commit message: get camera holder and fingers in hopefully good places

File: ur_e_description/urdf/ur5e.urdf.xacro (robot description, xacro)
@@ -334,5 +334,5 @@
       <parent link="${prefix}hand_link" />
       <child link = "${prefix}grasp_point_fixed" />
-      <origin xyz="0.0 0.0 0.050" rpy="0.0 0.0 0.0" />
+      <origin xyz="0.0 ${0.046 + 0.015} 0.0" rpy="0.0 0.0 ${-pi/2.0}" />
     </joint>
     <link name="${prefix}finger_l_link">
@@ -375,12 +375,12 @@
     </link>
     <joint name="${prefix}finger_l_fixed_joint" type="fixed">
-      <parent link="${prefix}hand_link" />
+      <parent link="${prefix}grasp_point_fixed" />
       <child link = "${prefix}finger_l_link" />
-      <origin xyz="0.0 ${0.046 + 0.015} 0.0" rpy="0.0 0.0 ${-pi/2.0}" />
+      <origin xyz="0.0 0.0 0.0" rpy="0.0 0.0 0.0" />
     </joint>
     <joint name="${prefix}finger_r_fixed_joint" type="fixed">
-      <parent link="${prefix}hand_link" />
+      <parent link="${prefix}grasp_point_fixed" />
       <child link = "${prefix}finger_r_link" />
-      <origin xyz="0.0 ${0.046 + 0.015} 0.0" rpy="${pi} 0.0 ${-pi/2.0}" />
+      <origin xyz="0.0 0.0 0.0" rpy="${pi} 0.0 0.0" />
     </joint>
     <joint name="${prefix}ee_fixed_joint" type="fixed">
@@ -416,7 +416,7 @@
     </link>
     <joint name="${prefix}camera_holder_fixed_joint" type="fixed">
-      <parent link="${prefix}wrist_3_link" />
+      <parent link="${prefix}hand_link" />
       <child link = "${prefix}camera_holder" />
-      <origin xyz="0.0 0.0 0.0" rpy="0.0 0.0 0.0" />
+      <origin xyz="0.0315 -0.001 0.0" rpy="${-pi/2} ${-pi/2} 0.0" />
     </joint>
     <xacro:ur_arm_transmission prefix="${prefix}" />

Commit message: add camera

File: ur_e_description/urdf/ur5e.urdf.xacro (robot description, xacro)
@@ -440,4 +440,10 @@
       <child link="${prefix}tool0"/>
     </joint>
+    <!-- realsense camera -->
+    <xacro:include filename="$(find realsense2_camera)/urdf/_d435.urdf.xacro" />
+    <!-- see http://wiki.ros.org/xacro for an explanation of the syntax of starred parameter passing -->
+    <xacro:sensor_d435 parent="${prefix}camera_holder">
+      <origin xyz="0 0.02 -0.049" rpy="0 ${-pi/2 - 0.6106} ${-pi/2}"/>
+    </xacro:sensor_d435>
   </xacro:macro>
 </robot>

Commit message: add gripper joints

File: ur_e_description/urdf/ur5e.urdf.xacro (robot description, xacro)
@@ -374,13 +374,19 @@
       </xacro:cylinder_inertial>
     </link>
-    <joint name="${prefix}finger_l_fixed_joint" type="fixed">
+    <joint name="${prefix}finger_l_fixed_joint" type="prismatic">
       <parent link="${prefix}grasp_point_fixed" />
       <child link = "${prefix}finger_l_link" />
-      <origin xyz="0.0 0.0 0.0" rpy="0.0 0.0 0.0" />
-    </joint>
-    <joint name="${prefix}finger_r_fixed_joint" type="fixed">
+      <origin xyz="0.0 0.0 -0.0059" rpy="0.0 0.0 0.0" />
+      <limit lower="0" upper="0.020" effort="150.0" velocity="1.0"/>
+      <!-- align motion on z-axis to match vrep's expectation -->
+      <axis xyz="0 0 1"/>
+    </joint>
+    <joint name="${prefix}finger_r_fixed_joint" type="prismatic">
       <parent link="${prefix}grasp_point_fixed" />
       <child link = "${prefix}finger_r_link" />
-      <origin xyz="0.0 0.0 0.0" rpy="${pi} 0.0 0.0" />
+      <origin xyz="0.0 0.0 0.0059" rpy="${pi} 0.0 0.0" />
+      <limit lower="0" upper="0.020" effort="150.0" velocity="1.0"/>
+      <!-- align motion on z-axis to match vrep's expectation -->
+      <axis xyz="0 0 1"/>
     </joint>
     <joint name="${prefix}ee_fixed_joint" type="fixed">

Commit message: rename to joint not fixed_joint

File: ur_e_description/urdf/ur5e.urdf.xacro (robot description, xacro)
@@ -374,5 +374,5 @@
       </xacro:cylinder_inertial>
     </link>
-    <joint name="${prefix}finger_l_fixed_joint" type="prismatic">
+    <joint name="${prefix}finger_l_joint" type="prismatic">
       <parent link="${prefix}grasp_point_fixed" />
       <child link = "${prefix}finger_l_link" />
@@ -382,5 +382,5 @@
       <axis xyz="0 0 1"/>
     </joint>
-    <joint name="${prefix}finger_r_fixed_joint" type="prismatic">
+    <joint name="${prefix}finger_r_joint" type="prismatic">
       <parent link="${prefix}grasp_point_fixed" />
       <child link = "${prefix}finger_r_link" />

Commit message: simplify xacro so we can use it with moveit directly with no collisions

File: ur_e_description/urdf/ur5e.urdf.xacro (robot description, xacro)
@@ -278,29 +278,4 @@
       </xacro:cylinder_inertial>
     </link>
-    <link name="${prefix}wrist_coupling_link">
-      <visual>
-        <geometry>
-          <mesh filename="package://ur_e_description/meshes/ur5e/visual/wrist_coupling.STL" />
-        </geometry>
-        <material name="LightGrey">
-          <color rgba="0.7 0.7 0.7 1.0"/>
-        </material>
-      </visual>
-      <collision>
-        <geometry>
-          <mesh filename="package://ur_e_description/meshes/ur5e/visual/wrist_coupling.STL" />
-        </geometry>
-      </collision>
-      <!-- computed from https://robotiq.com/support/hand-e-adaptive-robot-gripper/documents-gripper-instruction-manual-e-series weight was guessed -->
-      <xacro:cylinder_inertial radius="0.375" length="0.0169" mass="0.010">
-        <origin xyz="0.0 0.0 0.0" rpy="0 0 0" />
-      </xacro:cylinder_inertial>
-    </link>
-    <joint name="${prefix}wrist_coupling_fixed_joint" type="fixed">
-      <parent link="${prefix}wrist_3_link" />
-      <child link = "${prefix}wrist_coupling_link" />
-      <!-- will need to fudge the length to account for origin being inside the coupling -->
-      <origin xyz="0.0 ${wrist_3_length} 0.0" rpy="${-pi/2.0} 0.0 0.0" />
-    </joint>
     <link name="${prefix}hand_link">
       <visual>
@@ -324,9 +299,9 @@
       </inertial>
     </link>
-    <joint name="${prefix}hand_coupling_fixed_joint" type="fixed">
-      <parent link="${prefix}wrist_coupling_link" />
+    <joint name="${prefix}hand_wrist_fixed_joint" type="fixed">
+      <parent link="${prefix}wrist_3_link" />
       <child link = "${prefix}hand_link" />
       <!-- we fudge the length to make the two line up (probably because origin of hand is in rando place -->
-      <origin xyz="0.0 0.0 ${0.1005 - 0.0075}" rpy="${pi/2.0} 0.0 ${pi/2.0}" />
+      <origin xyz="0.0 ${wrist_3_length + 0.1005 - 0.0075} 0.0" rpy="0.0 ${-pi/2.0} 0.0" />
     </joint>
     <link name="${prefix}grasp_point_fixed"/>
@@ -446,10 +421,4 @@
       <child link="${prefix}tool0"/>
     </joint>
-    <!-- realsense camera -->
-    <xacro:include filename="$(find realsense2_camera)/urdf/_d435.urdf.xacro" />
-    <!-- see http://wiki.ros.org/xacro for an explanation of the syntax of starred parameter passing -->
-    <xacro:sensor_d435 parent="${prefix}camera_holder">
-      <origin xyz="0 0.02 -0.049" rpy="0 ${-pi/2 - 0.6106} ${-pi/2}"/>
-    </xacro:sensor_d435>
   </xacro:macro>
 </robot>
